File: lemon-microcontroller/lemon-pcb.kicad_pcb (KiCad board)
At the start: 2 copper layers, 31.9 x 36 mm, 52 parts, among them J1 USB_C_Receptacle_USB2.0, J2 USB_C_Receptacle_USB2.0, J3 Conn_01x11, J5 Conn_01x11, Q1 Q_NMOS, Q2 Q_PMOS_SGD, SW1 SW_Push, SW2 SW_Push, U1 W25Q128JVS, U2 USBLC6-2SC6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

Commit message: Update Wired Lemon V03 information
Parts:
- removed R15: 5k1, Resistor_SMD:R_0402_1005Metric
- added G***: LOGO, LOGO, F.Cu at (184.3, 50.7)
- added G***: LOGO, LOGO, B.Cu at (190.3, 47.2)
- added svg2mod: G***, Footprints:cosmoslogo-kicad-small, B.Cu at (194.4, 64.0)
- moved R14 0.48 mm to (183.4, 57.0), turned to 90 degrees
Connections:
- J3 pad 6: /GPIO27 -> VIK_GP2
- J3 pad 7: VIK_GP2 -> VIK_GP1
- U3 pad 27: VIK_GP1 -> unconnected-(U3-GPIO16-Pad27)
- U3 pad 38: VIK_GP2 -> VIK_GP1
- U3 pad 39: /GPIO27 -> VIK_GP2
Routing:
- net VIK_GP1: track 23.7 -> 44.5 mm, vias 2 -> 3
- net /GPIO27: track 10.5 -> 0.00 mm, vias 1 -> 0
- net +5V: track 96.7 -> 92.8 mm
- net GND: track 101.3 -> 104.2 mm
- net +3V3: track 94.4 -> 92.1 mm
- net /GPIO2: track 25.5 -> 24.0 mm
- net VIK_GP2: track 39.2 -> 40.0 mm
Other:
- board text added: "A Cosmos Project"

Commit message: Lemon wired V0.4, Lemon wireless V0.3
Parts:
- FPC1: footprint FPC-SMD_21P-P0.30_HDGC_0.3K-QX-21PWB -> Footprints:FPC-SMD_21P-P0.30_HDGC_0.3K-QX-21PWB
- FPC2: footprint ProPrj_New-easyedapro:FPC-SMD_10P-P0.50_HC-FPC-05-09-10RLTAG -> Footprints:FPC-SMD_10P-P0.50_HC-FPC-05-09-10RLTAG
- U1: value W25Q128JVS -> ZD25WQ80CTIGT; footprint Package_SO:SOP-8_3.9x4.9mm_P1.27mm -> Package_SO:SOIC-8_3.9x4.9mm_P1.27mm
- U4: value XC6206PxxxMR-Regulator_Linear -> XC6206P332MR-G
- VIK1: footprint ProPrj_New-easyedapro:FPC-SMD_FPC05012-09200 -> Footprints:FPC-SMD_FPC05012-09200
Connections:
- net /GPIO2 renamed /RGB
- FPC1 pad 10: /GPIO4 -> /R4
- FPC1 pad 11: /GPIO9 -> /R3
- FPC1 pad 12: /GPIO6 -> /R2
- FPC1 pad 13: /GPIO10 -> /R1
- FPC1 pad 8: /GPIO5 -> /R6
- FPC1 pad 9: /GPIO8 -> /R5
- FPC2 pad 1: /GPIO3 -> /R7
- J5 pad 10: /GPIO9 -> /R7
- J5 pad 11: /GPIO10 -> /C7
- J5 pad 4: /GPIO3 -> /R1
- J5 pad 5: /GPIO4 -> /R2
- J5 pad 6: /GPIO5 -> /R3
- J5 pad 7: /GPIO6 -> /R4
- J5 pad 8: /C7 -> /R5
- J5 pad 9: /GPIO8 -> /R6
- U3 pad 11: /GPIO8 -> /R6
- U3 pad 12: /GPIO9 -> /R7
- U3 pad 13: /GPIO10 -> /C7
- U3 pad 5: /GPIO3 -> /R1
- U3 pad 6: /GPIO4 -> /R2
- U3 pad 7: /GPIO5 -> /R3
- U3 pad 8: /GPIO6 -> /R4
- U3 pad 9: /C7 -> /R5
Routing:
- net /R3: track 0.00 -> 56.9 mm, vias 0 -> 3
- net /GPIO3: track 56.3 -> 0.00 mm, vias 2 -> 0
- net /R1: track 0.00 -> 54.1 mm, vias 0 -> 2
- net /GPIO5: track 53.3 -> 0.00 mm, vias 1 -> 0
- net /R7: track 0.00 -> 49.5 mm, vias 0 -> 1
- net /R2: track 0.00 -> 49.2 mm, vias 0 -> 2
- net /GPIO4: track 48.9 -> 0.00 mm, vias 2 -> 0
- net /R5: track 0.00 -> 46.0 mm, vias 0 -> 1
- net /GPIO6: track 45.9 -> 0.00 mm, vias 2 -> 0
- net /R4: track 0.00 -> 45.4 mm, vias 0 -> 2
- net /R6: track 0.00 -> 43.9 mm, vias 0 -> 1
- net /GPIO8: track 42.9 -> 0.00 mm, vias 1 -> 0
- net /GPIO9: track 42.1 -> 0.00 mm, vias 1 -> 0
- net /GPIO10: track 42.0 -> 0.00 mm, vias 1 -> 0
- net GND: track 104.2 -> 96.7 mm, vias 33 -> 32
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- added copper zone on F.Cu, net +5V
Other:
- board text added: "VIK OUT"
