File: lemon-wireless-uc/lemon-pcb-wireless.kicad_pcb (KiCad board)
At the start: 4 copper layers, 29.9 x 42 mm, 41 parts, among them J1 USB_C_Receptacle_USB2.0, J2 Conn_01x02, J3 Conn_01x11, J4 Programmer, J5 Conn_01x11, Q1 Q_NMOS, Q2 Q_PMOS_SGD, SW1 SW_SPDT_312, SW2 SW_Push, U1 74HC595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

Commit message: Lemon wired V0.4, Lemon wireless V0.3
Parts:
- removed R15: 5k1, Resistor_SMD:R_0402_1005Metric
- removed R9: 10k, Resistor_SMD:R_0402_1005Metric
- added G***: LOGO, LOGO, F.Cu at (182.9, 38.1)
- added G***: LOGO, LOGO, B.Cu at (185.8, 61.3)
- added G***: cosmoslogo, Footprints:cosmoslogo-kicad-small, B.Cu at (193.6, 69.4)
- added JP4: SolderJumper_2_Bridged, Jumper:SolderJumper-2_P1.3mm_Bridged_Pad1.0x1.5mm, B.Cu at (186.7, 41.0)
- added TP1: TestPoint, TestPoint:TestPoint_THTPad_D1.0mm_Drill0.5mm, F.Cu at (200.1, 43.1)
- added TP2: TestPoint, TestPoint:TestPoint_THTPad_D1.0mm_Drill0.5mm, F.Cu at (200.1, 40.9)
- added svg2mod: G***, lemonlib:vik_small, F.Cu at (200.9, 63.9)
- C16, C17: footprint Capacitor_SMD:C_0402_1005Metric -> Capacitor_SMD:C_0603_1608Metric
- FPC1: footprint FPC-SMD_21P-P0.30_HDGC_0.3K-QX-21PWB -> Footprints:FPC-SMD_21P-P0.30_HDGC_0.3K-QX-21PWB
- FPC2: footprint ProPrj_New-easyedapro:FPC-SMD_10P-P0.50_HC-FPC-05-09-10RLTAG -> Footprints:FPC-SMD_10P-P0.50_HC-FPC-05-09-10RLTAG
- R1, R14: value 5k1 -> 10k
- VIK1: footprint ProPrj_New-easyedapro:FPC-SMD_FPC05012-09200 -> Footprints:FPC-SMD_FPC05012-09200
- moved C17 3.51 mm to (184.7, 60.6), turned to -90 degrees
- moved JP3 1.10 mm to (184.0, 41.0)
- moved JP1 0.81 mm to (189.2, 41.0), turned to -90 degrees
- moved U4 0.21 mm to (187.3, 61.0)
- moved C16 0.20 mm to (188.2, 63.5)
Connections:
- net /GPIO2 renamed /RGB
- D1 pad 4: +3V3 -> Net-(D1-VDD)
- J3 pad 10: /R3 -> /R5
- J3 pad 11: /R5 -> /R6
- J3 pad 12: /R1 -> /R7
- J3 pad 4: VIK_GP2 -> VIK_GP1
- J3 pad 5: VIK_GP1 -> VIK_GP2
- J3 pad 6: /R7 -> /R1
- J3 pad 7: /R4 -> /R2
- J3 pad 8: /R6 -> /R3
- J3 pad 9: /R2 -> /R4
- JP1 pad 1: +3V3 -> Net-(JP1-A)
- JP1 pad 2: Net-(JP1-B) -> +3V3
- R16 pad 1: Net-(JP1-B) -> Net-(JP1-A)
- U3 pad 2: /R5 -> /R6
- U3 pad 21: /R7 -> /R1
- U3 pad 22: /R4 -> /R2
- U3 pad 23: /R6 -> /R3
- U3 pad 27: /R2 -> /R4
- U3 pad 28: /R3 -> /R5
- U3 pad 3: /R1 -> /R7
Routing:
- net LED_PWR: track 9.85 -> 43.2 mm, vias 2 -> 3
- net /LED_DATA: track 21.9 -> 40.2 mm, vias 1 -> 3
- net Net-(JP1-B): track 18.2 -> 0.00 mm, vias 1 -> 0
- net Net-(JP1-A): track 0.00 -> 17.9 mm, vias 0 -> 1
- net Net-(D1-VDD): track 0.00 -> 16.5 mm, vias 0 -> 2
- net /R5: track 78.1 -> 63.2 mm, vias 2 -> 1
- net VIK_GP2: track 61.3 -> 47.3 mm, vias 5 -> 2
- net /R2: track 67.6 -> 56.7 mm, vias 1 -> 5
- net +3V3: track 38.1 -> 30.7 mm, vias 8 -> 6
- net /R3: track 63.4 -> 56.2 mm
- net /R7: track 55.3 -> 49.4 mm, vias 4 -> 2
- net /R4: track 56.3 -> 61.8 mm, vias 5 -> 1
- net GND: track 49.9 -> 52.7 mm, vias 27 -> 28
- net SWDIO: track 12.2 -> 10.6 mm
- net VDDH: track 38.5 -> 37.4 mm
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- added copper zone on F.Cu, net LED_PWR
Other:
- board text added: "${REVISION}"
- board text added: ",RGB"
- board text added: "5V 3.3V GND 0.29 0.31 0.20 0.22 0.24 0.09 0.10 1.13 1.15 RST"
- board text added: "A Cosmos Project"
- board text added: "LEDS"
- board text added: "VIK OUT"
- board text added: "V_{RGB}"
- board text removed: "5V 3.3V GND 0.31 0.29 0.20 0.22 0.24 0.09 0.10 1.13 1.15 RST"
- board text removed: "LED"
- board text removed: "v0.2"

Commit message: Lemon Wireless v0.4
Parts:
- removed Q1: Q_NMOS, Package_TO_SOT_SMD:SOT-523
- removed R14: 10k, Resistor_SMD:R_0402_1005Metric
- removed svg2mod: G***, lemonlib:vik_small
- added C4: 100nF, Capacitor_SMD:C_0402_1005Metric, F.Cu at (193.0, 65.0)
- added C5: 100nF, Capacitor_SMD:C_0402_1005Metric, F.Cu at (194.0, 65.0)
- added R9: 100k, Resistor_SMD:R_0402_1005Metric, F.Cu at (190.8, 64.9)
- added U5: TXS0102DQE, Package_SON:X2SON-8_1.4x1mm_P0.35mm, F.Cu at (191.4, 66.3)
- R1: value 10k -> 100k
- moved R1 1.72 mm to (189.9, 66.3), turned to -90 degrees
- moved Q2 0.10 mm to (187.5, 65.9)
Connections:
- Q2 pad 1: LED_ON -> /LED_ON_5V
- R1 pad 1: LED_ON -> VDDH
- R1 pad 2: VPROG -> /LED_ON_5V
- VIK1 pad 6: VDDH -> LED_PWR
Routing:
- net LED_PWR: track 43.2 -> 58.2 mm, vias 3 -> 4
- net VDDH: track 37.4 -> 23.3 mm
- net GND: track 52.7 -> 60.4 mm, vias 28 -> 30
- net +3V3: track 30.7 -> 37.2 mm
- net /LED_DATA: track 40.2 -> 35.2 mm
- net /LED_ON_5V: track 0.00 -> 3.46 mm
- net VPROG: track 33.9 -> 32.1 mm, vias 5 -> 4
- net /RGB: track 13.3 -> 11.8 mm
- net SPI1_RX: track 22.1 -> 21.6 mm
