File: lemon-wireless-uc/lemon-pcb-wireless.kicad_sch (KiCad schematic)
At the start: 40 parts, among them J1 USB_C_Receptacle_USB2.0, J2 Conn_01x02, J3 Conn_01x11, J4 Programmer, J5 Conn_01x11, Q1 Q_NMOS, Q2 Q_PMOS_SGD, SW1 SW_SPDT_312, SW2 SW_Push, U1 74HC595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

Commit message: Lemon wired V0.4, Lemon wireless V0.3
Parts:
- removed R15: 5k1, Resistor_SMD:R_0402_1005Metric, symbol Device:R_Small
- added JP4: SolderJumper_2_Bridged, Jumper:SolderJumper-2_P1.3mm_Bridged_Pad1.0x1.5mm, symbol Jumper:SolderJumper_2_Bridged
- added TP1, TP2: TestPoint, TestPoint:TestPoint_THTPad_D1.0mm_Drill0.5mm, symbol Connector:TestPoint
- C16, C17: footprint Capacitor_SMD:C_0402_1005Metric -> Capacitor_SMD:C_0603_1608Metric; LCSC C52923 -> C15849
- D2: LCSC C7371898 -> C7496802
- D5: LCSC C7371898 -> C779448
- FPC1: footprint (none) -> Footprints:FPC-SMD_21P-P0.30_HDGC_0.3K-QX-21PWB
- FPC2: footprint ProPrj_New-easyedapro:FPC-SMD_10P-P0.50_HC-FPC-05-09-10RLTAG -> Footprints:FPC-SMD_10P-P0.50_HC-FPC-05-09-10RLTAG
- J1: symbol Connector:USB_C_Receptacle_USB2.0 -> Connector:USB_C_Receptacle_USB2.0_16P; LCSC C165948 -> C2927038
- Q1: symbol Device:Q_NMOS_GDS -> Transistor_FET:Q_NMOS_GDS; LCSC C8545 -> C7507460
- Q2: symbol Device:Q_PMOS_GSD -> Transistor_FET:Q_PMOS_GSD
- R1, R14: value 5k1 -> 10k; LCSC C25905 -> C25744
- VIK1: footprint ProPrj_New-easyedapro:FPC-SMD_FPC05012-09200 -> Footprints:FPC-SMD_FPC05012-09200; LCSC C479750 -> C19273928
Connections:
- net +3V3: now also JP1.2 (B), JP4.2 (B); no longer D1.4 (VDD), JP1.1 (A)
- net LED_DATA: now also TP1.1
- net LED_PWR: now also TP2.1
- net R1: now also J3.6 (Pin_6), U3.21 (P0.20*); no longer J3.12 (Pin_12), U3.3 (P1.15)
- net R2: now also J3.7 (Pin_7), U3.22 (P0.22*); no longer J3.9 (Pin_9), U3.27 (P0.09)
- net R3: now also J3.8 (Pin_8), U3.23 (P0.24*); no longer J3.10 (Pin_10), U3.28 (P0.10)
- net R4: now also J3.9 (Pin_9), U3.27 (P0.09); no longer J3.7 (Pin_7), U3.22 (P0.22*)
- net R5: now also J3.10 (Pin_10), U3.28 (P0.10); no longer J3.11 (Pin_11), U3.2 (P1.13)
- net R6: now also J3.11 (Pin_11), U3.2 (P1.13); no longer J3.8 (Pin_8), U3.23 (P0.24*)
- net R7: now also J3.12 (Pin_12), U3.3 (P1.15); no longer J3.6 (Pin_6), U3.21 (P0.20*)
- net VIK_GP1: now also J3.4 (Pin_4); no longer J3.5 (Pin_5)
- net VIK_GP2: now also J3.5 (Pin_5); no longer J3.4 (Pin_4)
- net at R16.1: now also JP1.1 (A); no longer JP1.2 (B)
- net GPIO2 renamed RGB
- new net: D1.4 (VDD), JP4.1 (A)
Other:
- note added: "Breakout Pins"
- note added: "Onboard LED"
- note added: "Power and Battery"
- note added: "Programming"
- note added: "RGB LED 5V Logic/Power"
- note added: "Shift Register"
- note added: "USB Comm"
- moved on the sheet: D1, J4, JP1, Q1, Q2, R1, R14, SW2

Commit message: Lemon Wireless v0.4
Parts:
- removed Q1: Q_NMOS, Package_TO_SOT_SMD:SOT-523, symbol Transistor_FET:Q_NMOS_GDS
- removed Q2: Q_PMOS_SGD, Package_TO_SOT_SMD:SOT-23, symbol Transistor_FET:Q_PMOS_GSD
- removed R14: 10k, Resistor_SMD:R_0402_1005Metric, symbol Device:R_Small
- added C4, C5: 100nF, Capacitor_SMD:C_0402_1005Metric, symbol Device:C_Small
- added Q2: Q_PMOS_SGD, Package_TO_SOT_SMD:SOT-23, symbol Device:Q_PMOS_GSD
- added R9: 100k, Resistor_SMD:R_0402_1005Metric, symbol Device:R_Small
- added U5: TXS0102DQE, Package_SON:X2SON-8_1.4x1mm_P0.35mm, symbol Logic_LevelTranslator:TXS0102DQE
- FPC1: LCSC C2919509 -> C3012330
- J1: LCSC C2927038 -> C165948
- J3, J5, TP1, TP2: now left out of the parts list
- R1: value 10k -> 100k; LCSC C25744 -> C25741
- SW1: FT Position Offset (none) -> 0,0.381
- U1: FT Rotation Offset (none) -> -90
Connections:
- net GND: now also C4.1, C5.1, R9.2, U5.3 (A2), U5.4 (GND)
- net LED_DATA: now also U5.7 (B1)
- net LED_ON: now also R9.1, U5.5 (OE); no longer R1.1
- net LED_PWR: now also VIK1.6 (Pin_6), Q2.3 (D)
- net RGB: now also U5.2 (A1)
- net VDDH: now also R1.1, C5.2, Q2.2 (S), U5.8 (VCCB); no longer VIK1.6 (Pin_6)
- net VPROG: now also C4.2, U5.1 (VCCA); no longer R1.2
- new net LED_ON_5V: Q2.1 (G), R1.2, U5.6 (B2)
